Commit message: multiple objects and color pick

File: assets/objects/cuboid0.urdf (robot description, URDF)
Before this commit: robot cuboid0, 1 links, 0 joints
Links:
- link baseLink: geometry collision mesh filename=cuboid0.obj; visual mesh filename=cuboid0.obj

File: assets/objects/cuboid1.urdf (robot description, URDF)
Before this commit: robot triangle, 1 links, 0 joints
Links:
- link baseLink: mass 0.020 -> 0.025; geometry collision mesh filename=cuboid1.obj; visual mesh filename=cuboid1.obj

File: assets/objects/custom.urdf (robot description, URDF)
Before this commit: robot custom, 1 links, 0 joints
Links:
- link base_link: geometry collision mesh filename=custom.obj scale=1 1 1; visual mesh filename=custom.obj scale=1 1 1

File: assets/objects/cylinder.urdf (robot description, URDF)
Before this commit: robot cylinder, 1 links, 0 joints
Links:
- link baseLink: geometry collision mesh filename=cylinder.obj; visual mesh filename=cylinder.obj

File: assets/objects/triangle.urdf (robot description, URDF)
Before this commit: robot cuboid1, 1 links, 0 joints
Links:
- link baseLink: mass 0.025 -> 0.020; geometry collision mesh filename=triangle.obj; visual mesh filename=triangle.obj
